File: KicadV6/Pico_Interface.kicad_sch (KiCad schematic)
At the start: 11 parts, among them J0 Conn_02x06_Odd_Even, J1 Conn_02x06_Odd_Even, J2 Conn_02x06_Odd_Even, J3 Conn_02x06_Odd_Even, J4 Conn_01x03_Male, J5 Conn_01x02_Male, J6 Conn_01x03_Male, J7 Conn_01x02_Male, U1 Pico, U2 NCP1117-3.3_SOT223

Commit message: Added Title Block
Other:
- company: (none) -> CERN Magnus Mager & USN 
- title: (none) -> Pico Readout for ITS Outer Barrel Model
Changed lines of the file:
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@@
 (kicad_sch (version 20211123) (generator eeschema)
   (paper "A4")
+  (title_block
+    (title "Pico Readout for ITS Outer Barrel Model")
+    (date "2022-10-21")
+    (rev "V0.1")
+    (company "CERN Magnus Mager & USN ")
+  )
   (junction (at 74.93 115.57) (diameter 0) (color 0 0 0 0)
   )
